Commit message: update

File: aljnu_description/urdf/aljnu_mp.urdf.xacro (robot description, xacro)
@@ -7,8 +7,8 @@
     <!-- Include middle box -->
     <xacro:include filename="$(find aljnu_description)/urdf/middle_box.urdf.xacro" />
-    <!-- Include robotiq85 -->
+    <!-- Include robotiq85 adapter -->
     <xacro:include filename="$(find aljnu_description)/urdf/robotiq85/ur_to_robotiq_adapter.urdf.xacro" />
-    <!-- Attach Gripper to UR5e -->
     <xacro:ur_to_robotiq prefix="" connected_to="ur5e_tool0" rotation="0.0" />
+    <!-- Include robotiq85 gripper -->
     <xacro:include filename="$(find aljnu_description)/urdf/robotiq85/robotiq_85_macro.urdf.xacro" />
     <xacro:robotiq_85_gripper prefix="" parent="gripper_mount_link">

File: aljnu_description/urdf/robotiq85/robotiq_85_macro.urdf.xacro (robot description, xacro)
@@ -8,6 +8,25 @@
 		</joint>
 		<link name="${prefix}robotiq_85_base_link">
-			<visual>
-				<origin xyz="0.16 0 0" rpy="0 0 0" />
+			<visual> <!-- Gripper body -->
+				<geometry>
+					<mesh filename="package://aljnu_description/meshes/robotiq85/visual/robotiq_85_base_link.dae"/>
+				</geometry>
+			</visual>
+			<collision>
+				<geometry>
+					<mesh filename="package://aljnu_description/meshes/robotiq85/collision/robotiq_85_base_link.stl"/>
+				</geometry>
+			</collision>
+			<inertial>
+				<mass value="0.636951" />
+				<origin xyz="0.0 0.0 0.0" />
+				<inertia ixx = "0.000380" ixy = "0.000000" ixz = "0.000000"
+					iyx = "0.000000" iyy = "0.001110" iyz = "0.000000"
+					izx = "0.000000" izy = "0.000000" izz = "0.001171" />
+			</inertial>
+		</link>
+		<link name="${prefix}robotiq_85_tip">
+			<visual>
+				<origin xyz="0 0 0" rpy="0 0 0" />
 				<geometry>
 					<sphere radius="0.007"/> <!-- Visual aid for grasping sphere in front of gripper -->
@@ -17,22 +36,10 @@
 				</material>
 			</visual>
-			<visual> <!-- Gripper body -->
-				<geometry>
-					<mesh filename="package://aljnu_description/meshes/robotiq85/visual/robotiq_85_base_link.dae"/>
-				</geometry>
-			</visual>
-			<collision>
-				<geometry>
-					<mesh filename="package://aljnu_description/meshes/robotiq85/collision/robotiq_85_base_link.stl"/>
-				</geometry>
-			</collision>
-			<inertial>
-				<mass value="0.636951" />
-				<origin xyz="0.0 0.0 0.0" />
-				<inertia ixx = "0.000380" ixy = "0.000000" ixz = "0.000000"
-					iyx = "0.000000" iyy = "0.001110" iyz = "0.000000"
-					izx = "0.000000" izy = "0.000000" izz = "0.001171" />
-			</inertial>
-		</link>
+		</link>
+		<joint name="${prefix}robotiq_85_base_to_tip_joint" type="fixed">
+			<parent link="${prefix}robotiq_85_base_link"/>
+			<child link="${prefix}robotiq_85_tip"/>
+			<origin xyz="0.16 0 0" rpy="0 0 0" />
+		</joint>
 		<joint name="${prefix}robotiq_85_left_knuckle_joint" type="revolute">
 			<parent link="${prefix}robotiq_85_base_link"/>

File: aljnu_description/urdf/ur5e/ur.urdf.xacro (robot description, xacro)
@@ -7,5 +7,5 @@
    <!-- possible 'ur_type' values: ur3, ur3e, ur5, ur5e, ur10, ur10e, ur16e, ur20, ur30 -->
    <!-- the default value should raise an error in case this was called without defining the type -->
-   <xacro:arg name="ur_type" default="ur5x"/>
+   <xacro:arg name="ur_type" default="ur5e"/>
    <!-- parameters -->
    <xacro:arg name="tf_prefix" default="" />
